File: DMH_Multiverter_Mk2_PCB_Conn/DMH_Multiverter_Mk2_PCB_Conn.kicad_sch (KiCad schematic)
At the start: 0 parts

Commit message: pcb 2 in progress
Connections:
- no-connect marks 4 -> 6
Other:
- sheet Inputs and Outputs ports: added Att C Input Jack, Att C Output Jack; removed none
Changed lines of the file:
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@@
 	)
 	(no_connect
-		(at 38.1 101.6)
+		(at 38.1 93.98)
 	)
 	(no_connect
@@
 	)
 	(no_connect
-		(at 38.1 88.9)
+		(at 38.1 81.28)
+	)
+	(no_connect
+		(at 38.1 97.79)
 	)
 	(no_connect
 		(at 38.1 105.41)
+	)
+	(no_connect
+		(at 38.1 109.22)
 	)
 	(sheet
@@
 		)
 		(pin "Att B Output Jack" input
+			(at 38.1 97.79 0)
+			(effects
+				(font
+					(size 1.27 1.27)
+				)
+				(justify right)
+			)
+		)
+		(pin "Att B Input Jack" output
+			(at 38.1 93.98 0)
+			(effects
+				(font
+					(size 1.27 1.27)
+				)
+				(justify right)
+			)
+		)
+		(pin "Att A Input Jack" output
+			(at 38.1 81.28 0)
+			(effects
+				(font
+					(size 1.27 1.27)
+				)
+				(justify right)
+			)
+		)
+		(pin "Att A Output Jack" input
+			(at 38.1 85.09 0)
+			(effects
+				(font
+					(size 1.27 1.27)
+				)
+				(justify right)
+			)
+		)
+		(pin "Att C Input Jack" output
 			(at 38.1 105.41 0)
 			(effects
@@
 			)
 		)
-		(pin "Att B Input Jack" output
-			(at 38.1 101.6 0)
-			(effects
-				(font
-					(size 1.27 1.27)
-				)
-				(justify right)
-			)
-		)
-		(pin "Att A Input Jack" output
-			(at 38.1 85.09 0)
-			(effects
-				(font
-					(size 1.27 1.27)
-				)
-				(justify right)
-			)
-		)
-		(pin "Att A Output Jack" input
-			(at 38.1 88.9 0)
+		(pin "Att C Output Jack" input
+			(at 38.1 109.22 0)
 			(effects
 				(font
@@
 		)
 		(instances
-			(project "DMH_Multiverter_PCB_Conn"
+			(project "DMH_Multiverter_Mk2_PCB_Conn"
 				(path "/58f4306d-5387-4983-bb08-41a2313fd315"
 					(page "2")
