File: DMH_Multiverter_Mk2_PCB_Conn/DMH_Multiverter_Mk2_PCB_Conn.kicad_pcb (KiCad board)
At the start: 2 copper layers, 48 x 175 mm, 24 parts, among them J1 TS_Jack_6.35mm_Sw, J10 TS_Jack_6.35mm_Sw, J11 TS_Jack_6.35mm_Sw, J12 TS_Jack_6.35mm_Sw, J13 TS_Jack_6.35mm_Sw, J14 TS_Jack_6.35mm_Sw, J15 TS_Jack_6.35mm_Sw, J16 TS_Jack_6.35mm_Sw, J17 TS_Jack_6.35mm_Sw, J18 TS_Jack_6.35mm_Sw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

Commit message: pcb 2 in progress
Parts:
- removed J16, J17, J18, J19, J20, J21, J22: TS_Jack_6.35mm_Sw, SynthStuff:CUI_MJ-63052A
- J50, J60: value Conn_01x06 -> Conn_01x08; footprint Connector_PinHeader_2.54mm:PinHeader_1x06_P2.54mm_Vertical -> Connector_PinHeader_2.54mm:PinHeader_1x08_P2.54mm_Vertical
- moved J10 59.5 mm to (58.5, 192.2), turned to -90 degrees
- moved J13 59.5 mm to (58.5, 208.8), turned to -90 degrees
- moved J11 36.9 mm to (75.0, 192.2), turned to 0 degrees
- moved J12 36.9 mm to (91.5, 192.2), turned to 90 degrees
- moved J14 36.9 mm to (75.0, 208.8), turned to 0 degrees
- moved J15 36.9 mm to (91.5, 208.8), turned to 90 degrees
Connections:
- J10 pad TN: unconnected-(J10-PadTN) -> Net-(J10-PadTN)
- J11 pad T: Net-(J11-PadT) -> Net-(J10-PadT)
- J11 pad TN: Net-(J10-PadT) -> unconnected-(J11-PadTN)
- J12 pad T: Net-(J11-PadT) -> Net-(J10-PadT)
- J13 pad T: Net-(J11-PadT) -> Net-(J13-PadT)
- J13 pad TN: unconnected-(J13-PadTN) -> Net-(J10-PadT)
- J14 pad T: Net-(J14-PadT) -> Net-(J13-PadT)
- J14 pad TN: Net-(J11-PadT) -> unconnected-(J14-PadTN)
- J15 pad T: Net-(J14-PadT) -> Net-(J13-PadT)
- J3 pad TN: Net-(J60-Pin_3) -> Net-(J60-Pin_1)
- J5 pad T: Net-(J5-PadT) -> /Inputs and Outputs/Att C Input Jack
- J5 pad TN: unconnected-(J5-PadTN) -> Net-(J60-Pin_1)
- J50 pad 5: GND -> /Inputs and Outputs/Att C Input Jack
- J50 pad 6: GND -> /Inputs and Outputs/Att C Output Jack
- J6 pad T: Net-(J5-PadT) -> /Inputs and Outputs/Att C Output Jack
- J6 pad TN: unconnected-(J6-PadTN) -> Net-(J60-Pin_6)
- J60 pad 3: Net-(J60-Pin_3) -> Net-(J60-Pin_1)
- J60 pad 5: GND -> Net-(J60-Pin_1)
- J60 pad 6: GND -> Net-(J60-Pin_6)
- J7 pad T: Net-(J5-PadT) -> Net-(J10-PadTN)
- J8 pad T: Net-(J10-PadT) -> Net-(J10-PadTN)
- J8 pad TN: Net-(J5-PadT) -> unconnected-(J8-PadTN)
- J9 pad T: Net-(J10-PadT) -> Net-(J10-PadTN)
Routing:
- net Net-(J10-PadTN): track 0.00 -> 108.3 mm
- net Net-(J17-PadT): track 54.3 -> 0.00 mm
- net Net-(J10-PadT): track 54.1 -> 108.4 mm
- net Net-(J14-PadT): track 54.1 -> 0.00 mm
- net Net-(J11-PadT): track 54.1 -> 0.00 mm
- net Net-(J5-PadT): track 53.8 -> 0.00 mm
- net (no net): track 0.00 -> 53.8 mm
- net Net-(J60-Pin_1): track 108.0 -> 147.9 mm
- net Net-(J60-Pin_3): track 39.9 -> 0.00 mm
- net Net-(J20-PadT): track 39.3 -> 0.00 mm
- net Net-(J13-PadT): track 0.00 -> 39.3 mm

Commit message: Routed Connectors PCB
Parts:
- J50, J60: footprint Connector_PinHeader_2.54mm:PinHeader_1x08_P2.54mm_Vertical -> Connector_PinSocket_2.54mm:PinSocket_1x08_P2.54mm_Vertical
- moved J7 59.5 mm to (58.5, 175.8), turned to 0 degrees
- moved J60 49.6 mm to (92.4, 165.0)
- moved J8 36.9 mm to (75.0, 175.8), turned to 0 degrees
- moved J9 36.9 mm to (91.5, 175.8), turned to 90 degrees
- moved J6 23.9 mm to (58.5, 143.5)
- moved J50 20.8 mm to (69.0, 92.0)
- moved J5 0.25 mm to (58.5, 126.5), turned to 0 degrees
- turned J10 to 0 degrees
- turned J13 to 0 degrees
- turned J2 to 0 degrees
- turned J3 to 0 degrees
- turned J4 to 0 degrees
Routing:
- net Net-(J60-Pin_4): track 24.2 -> 91.5 mm
- net Net-(J10-PadT): track 108.4 -> 41.4 mm
- net Net-(J10-PadTN): track 108.3 -> 41.4 mm
- net (no net): track 53.8 -> 0.00 mm
- net Net-(J60-Pin_6): track 0.00 -> 46.2 mm
- net Net-(J60-Pin_2): track 86.6 -> 126.8 mm
- net /Inputs and Outputs/Att C Output Jack: track 0.00 -> 40.0 mm
- net /Inputs and Outputs/Att B Output Jack: track 37.1 -> 6.79 mm
- net /Inputs and Outputs/Att C Input Jack: track 0.00 -> 25.5 mm
- net /Inputs and Outputs/Att A Output Jack: track 10.1 -> 30.7 mm
- net /Inputs and Outputs/Att A Input Jack: track 21.3 -> 39.6 mm
- net /Inputs and Outputs/Att B Input Jack: track 25.7 -> 11.0 mm
- net Net-(J13-PadT): track 39.3 -> 29.2 mm
- net Net-(J60-Pin_1): track 147.9 -> 156.5 mm
Other:
- outline, holes or cut-outs redrawn
- board text added: "Mk2.0 - March 2025"
- board text removed: "Mk1.0 - December 2024"

Commit message: Independent zeners for normalled 5V DC offset
Connections:
- J3 pad TN: Net-(J60-Pin_1) -> Net-(J60-Pin_3)
- J5 pad TN: Net-(J60-Pin_1) -> Net-(J60-Pin_5)
- J60 pad 3: Net-(J60-Pin_1) -> Net-(J60-Pin_3)
- J60 pad 5: Net-(J60-Pin_1) -> Net-(J60-Pin_5)
Routing:
- net Net-(J60-Pin_3): track 0.00 -> 113.5 mm
- net Net-(J60-Pin_5): track 0.00 -> 66.7 mm
- net Net-(J60-Pin_1): track 156.5 -> 158.3 mm
Changed lines of the file:
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@@
 	(net 20 "unconnected-(J15-PadTN)")
 	(net 21 "unconnected-(J14-PadTN)")
+	(net 22 "Net-(J60-Pin_3)")
+	(net 23 "Net-(J60-Pin_5)")
 	(footprint "SynthStuff:CUI_MJ-63052A"
 		(layer "F.Cu")
@@
 			(layers "*.Cu" "*.Mask")
 			(remove_unused_layers no)
-			(net 2 "Net-(J60-Pin_1)")
+			(net 22 "Net-(J60-Pin_3)")
 			(pinfunction "Pin_3")
 			(pintype "passive")
@@
 			(layers "*.Cu" "*.Mask")
 			(remove_unused_layers no)
-			(net 2 "Net-(J60-Pin_1)")
+			(net 23 "Net-(J60-Pin_5)")
 			(pinfunction "Pin_5")
 			(pintype "passive")
@@
 			(layers "*.Cu" "*.Mask")
 			(remove_unused_layers no)
-			(net 2 "Net-(J60-Pin_1)")
+			(net 23 "Net-(J60-Pin_5)")
 			(pintype "passive")
 			(solder_mask_margin 0.102)
@@
 			(layers "*.Cu" "*.Mask")
 			(remove_unused_layers no)
-			(net 2 "Net-(J60-Pin_1)")
+			(net 22 "Net-(J60-Pin_3)")
 			(pintype "passive")
 			(solder_mask_margin 0.102)
@@
 	)
 	(segment
-		(start 87.295 164.975)
-		(end 85.77 166.5)
-		(width 0.2)
-		(layer "F.Cu")
-		(net 2)
-	)
-	(segment
-		(start 92.375 164.975)
-		(end 90.85 166.5)
-		(width 0.2)
-		(layer "F.Cu")
-		(net 2)
-	)
-	(segment
-		(start 83.74 166.5)
-		(end 82.215 164.975)
-		(width 0.2)
-		(layer "F.Cu")
-		(net 2)
-	)
-	(segment
-		(start 90.85 166.5)
-		(end 88.82 166.5)
-		(width 0.2)
-		(layer "F.Cu")
-		(net 2)
-	)
-	(segment
-		(start 85.77 166.5)
-		(end 83.74 166.5)
-		(width 0.2)
-		(layer "F.Cu")
-		(net 2)
-	)
-	(segment
-		(start 88.82 166.5)
-		(end 87.295 164.975)
+		(start 57.227376 52.5)
+		(end 65 52.5)
 		(width 0.2)
-		(layer "F.Cu")
+		(layer "B.Cu")
 		(net 2)
 	)
 	(segment
-		(start 59.9 52.5)
-		(end 65 52.5)
+		(start 68.7678 168.902)
+		(end 57.988 158.1222)
 		(width 0.2)
 		(layer "B.Cu")
@@
 	)
 	(segment
-		(start 69.2661 167.699)
-		(end 59.191 157.6239)
+		(start 57.988 61.238)
+		(end 55 58.25)
 		(width 0.2)
 		(layer "B.Cu")
@@
 	)
 	(segment
-		(start 59.191 157.6239)
-		(end 59.191 121.809)
+		(start 74.239058 168.902)
+		(end 68.7678 168.902)
 		(width 0.2)
 		(layer "B.Cu")
@@
 	)
 	(segment
-		(start 59.191 121.809)
-		(end 61 120)
+		(start 91.224 166.126)
+		(end 87.77176 166.126)
 		(width 0.2)
 		(layer "B.Cu")
@@
 	)
 	(segment
-		(start 62.809 83.559)
-		(end 61 81.75)
+		(start 55 58.25)
+		(end 55 54.727376)
 		(width 0.2)
 		(layer "B.Cu")
@@
 	)
 	(segment
-		(start 79.491 167.699)
-		(end 69.2661 167.699)
+		(start 83.19176 170.706)
+		(end 76.043057 170.706)
 		(width 0.2)
 		(layer "B.Cu")
@@
 	)
 	(segment
-		(start 61 120)
-		(end 62.809 118.191)
+		(start 65 53.254)
+		(end 65 52.5)
 		(width 0.2)
 		(layer "B.Cu")
@@
 	)
 	(segment
-		(start 62.809 118.191)
-		(end 62.809 83.559)
+		(start 92.375 164.975)
+		(end 91.224 166.126)
 		(width 0.2)
 		(layer "B.Cu")
@@
 	)
 	(segment
-		(start 82.215 164.975)
-		(end 79.491 167.699)
+		(start 87.77176 166.126)
+		(end 83.19176 170.706)
 		(width 0.2)
 		(layer "B.Cu")
@@
 	)
 	(segment
-		(start 56.8 55.6)
-		(end 59.9 52.5)
+		(start 76.043057 170.706)
+		(end 74.239058 168.902)
 		(width 0.2)
 		(layer "B.Cu")
@@
 	)
 	(segment
-		(start 61 81.75)
-		(end 56.8 77.55)
+		(start 57.988 158.1222)
+		(end 57.988 61.238)
 		(width 0.2)
 		(layer "B.Cu")
@@
 	)
 	(segment
-		(start 56.8 77.55)
-		(end 56.8 55.6)
+		(start 55 54.727376)
+		(end 57.227376 52.5)
 		(width 0.2)
 		(layer "B.Cu")
@@
 	)
 	(segment
-		(start 58.79 157.79)
-		(end 58.79 119.21)
+		(start 58.79 100.96)
+		(end 61 98.75)
 		(width 0.2)
 		(layer "B.Cu")
@@
 	)
 	(segment
-		(start 58.79 119.21)
-		(end 61 117)
+		(start 58.79 157.79)
+		(end 58.79 100.96)
 		(width 0.2)
 		(layer "B.Cu")
@@
 	)
 	(segment
-		(start 69.1 168.1)
-		(end 58.79 157.79)
+		(start 84.755 164.975)
+		(end 81.63 168.1)
 		(width 0.2)
 		(layer "B.Cu")
@@
 	)
 	(segment
-		(start 61 117)
-		(end 61 98.75)
-		(width 0.2)
-		(layer "B.Cu")
-		(net 8)
-	)
-	(segment
-		(start 84.755 164.975)
-		(end 81.63 168.1)
+		(start 69.1 168.1)
+		(end 58.79 157.79)
 		(width 0.2)
 		(layer "B.Cu")
@@
 		(net 19)
 	)
+	(segment
+		(start 68.9339 168.501)
+		(end 58.389 157.9561)
+		(width 0.2)
+		(layer "B.Cu")
+		(net 22)
+	)
+	(segment
+		(start 74.405157 168.501)
+		(end 68.9339 168.501)
+		(width 0.2)
+		(layer "B.Cu")
+		(net 22)
+	)
+	(segment
+		(start 58.389 157.9561)
+		(end 58.389 84.361)
+		(width 0.2)
+		(layer "B.Cu")
+		(net 22)
+	)
+	(segment
+		(start 58.389 84.361)
+		(end 61 81.75)
+		(width 0.2)
+		(layer "B.Cu")
+		(net 22)
+	)
+	(segment
+		(start 81.965 170.305)
+		(end 76.209157 170.305)
+		(width 0.2)
+		(layer "B.Cu")
+		(net 22)
+	)
+	(segment
+		(start 87.295 164.975)
+		(end 81.965 170.305)
+		(width 0.2)
+		(layer "B.Cu")
+		(net 22)
+	)
+	(segment
+		(start 76.209157 170.305)
+		(end 74.405157 168.501)
+		(width 0.2)
+		(layer "B.Cu")
+		(net 22)
+	)
+	(segment
+		(start 82.215 164.975)
+		(end 79.491 167.699)
+		(width 0.2)
+		(layer "B.Cu")
+		(net 23)
+	)
+	(segment
+		(start 59.191 157.6239)
+		(end 59.191 121.809)
+		(width 0.2)
+		(layer "B.Cu")
+		(net 23)
+	)
+	(segment
+		(start 59.191 121.809)
+		(end 61 120)
+		(width 0.2)
+		(layer "B.Cu")
+		(net 23)
+	)
+	(segment
+		(start 79.491 167.699)
+		(end 69.2661 167.699)
+		(width 0.2)
+		(layer "B.Cu")
+		(net 23)
+	)
+	(segment
+		(start 69.2661 167.699)
+		(end 59.191 157.6239)
+		(width 0.2)
+		(layer "B.Cu")
+		(net 23)
+	)
 	(zone
